File: HW/DMX_CTRL/DMX_CTRL.kicad_pcb (KiCad board)
At the start: 2 copper layers, 50 x 100 mm, 43 parts, among them J1 LED_CONN, J10 TTL_UART, J2 MODE, J3 ADDR, J4 PWR, J5 12V Link, J6 WS2812_Conn, J7 AUX, J9 3V3 UART, Q1 IRLB8721PBF, Q10 IRLB8721PBF, Q2 IRLB8721PBF, Q3 IRLB8721PBF, Q4 IRLB8721PBF, Q5 IRLB8721PBF, Q6 IRLB8721PBF, Q7 IRLB8721PBF, Q8 IRLB8721PBF, Q9 IRLB8721PBF, SW1 SW_Push, U1 ChinaBluePill, U2 uA7805, U3 ESP-01, U4 RS485_Transeiver

Commit message: New PCB 2.0
Parts:
- removed H4: MountingHole, MountingHole:MountingHole_4.3mm_M4_DIN965_Pad
- added H3: MountingHole, MountingHole:MountingHole_4.3mm_M4_DIN965_Pad, F.Cu at (126.0, 146.0)
- added R13: 1K, Resistor_THT:R_Axial_DIN0204_L3.6mm_D1.6mm_P1.90mm_Vertical, F.Cu at (88.5, 72.4)
- added R14: 1K, Resistor_THT:R_Axial_DIN0204_L3.6mm_D1.6mm_P1.90mm_Vertical, F.Cu at (92.0, 72.4)
- added SW2: SW_Push, Button_Switch_THT:SW_PUSH_6mm_H8mm, F.Cu at (121.0, 142.0)
- Q1, Q10, Q2, Q3, Q4, Q5, Q6, Q7, Q8, Q9: value IRLB8721PBF -> IXTP3N50D2
- moved U4 41.6 mm to (94.0, 101.5), turned to 0 degrees
- moved U2 32.0 mm to (114.0, 69.0), turned to 180 degrees
- moved J5 27.6 mm to (115.5, 65.5), turned to -90 degrees
- moved C2 26.4 mm to (109.0, 74.0)
- moved C1 24.4 mm to (95.0, 72.5)
- moved C3 18.2 mm to (104.5, 86.0)
- moved J9 11.8 mm to (84.0, 72.0), turned to -90 degrees
- moved SW1 9.01 mm to (109.0, 148.5), turned to 90 degrees
- moved R12 6.95 mm to (104.0, 70.0)
- moved R11 6.79 mm to (104.0, 64.4)
- moved J10 4.68 mm to (86.5, 88.0)
- moved R8 1.93 mm to (108.5, 85.9), turned to 90 degrees
- moved R9 1.60 mm to (108.5, 91.4), turned to 90 degrees
- moved J6 1.45 mm to (75.0, 64.0)
- moved BT1 1.36 mm to (101.5, 56.8)
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Connections:
- J10 pad 2: /ADDR_1 -> Net-(J10-Pad2)
- J10 pad 4: /RS23_TX -> /RS232_RX
- J10 pad 5: /RS232_RX -> /RS23_TX
- J10 pad 6: /ADDR_0 -> Net-(J10-Pad6)
- U1 pad PA11: (no net) -> Net-(U1-PadPA11)
- U1 pad PA12: (no net) -> Net-(U1-PadPA12)
- U3 pad 2: /ADDR_0 -> Net-(J10-Pad6)
- U3 pad 3: /ADDR_1 -> Net-(J10-Pad2)
- U3 pad 6: (no net) -> +3V3
- U3 pad 7: /ADDR_2 -> +3V3
- U4 pad 5: (no net) -> GND
Routing:
- net Net-(J10-Pad2): track 0.00 -> 129.9 mm, vias 0 -> 1
- net /ADDR_0: track 98.4 -> 26.4 mm, vias 6 -> 3
- net /PWM_CH3_W: track 83.4 -> 24.5 mm, vias 2 -> 1
- net /ADDR_2: track 85.6 -> 34.7 mm, vias 5 -> 3
- net /RS485_A: track 71.0 -> 118.1 mm, vias 4 -> 1
- net /ADDR_1: track 83.2 -> 36.5 mm, vias 4 -> 2
- net +5V: track 130.4 -> 176.2 mm, vias 3 -> 4
- net /PWM_CH3_B: track 80.1 -> 35.2 mm, vias 4 -> 3
- net +12V: track 102.7 -> 68.4 mm
- net Net-(J6-Pad2): track 72.1 -> 41.9 mm, vias 3 -> 1
- net /RS485_B: track 88.1 -> 117.2 mm, vias 4 -> 0
- net /RS485_DIR: track 40.3 -> 15.5 mm
- net /ADDR_3: track 68.4 -> 44.4 mm
- net Net-(J10-Pad6): track 0.00 -> 19.9 mm
- net /RS485_RXTX: track 41.4 -> 23.1 mm, vias 1 -> 0
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Other:
- board text added: "1"
- board text added: "DMX_CTRL V2.0"
- board text added: "DMX_CTRL V2.0 (C) 2020 M. Hartmann"
- board text removed: "DMX_CTRL V1.0"
- board text removed: "DMX_CTRL V1.0 (C) 2020 M. Hartmann"
