File: HW/DMX_CTRL/_autosave-DMX_CTRL.kicad_pcb (KiCad board)
At the start: 2 copper layers, 50 x 100 mm, 46 parts, among them J1 LED_CONN, J10 TTL_UART, J2 MODE, J3 ADDR, J4 PWR, J5 12V Link, J6 WS2812_Conn, J7 AUX, J9 3V3 UART, Q1 IXTP3N50D2, Q10 IXTP3N50D2, Q2 IXTP3N50D2, Q3 IXTP3N50D2, Q4 IXTP3N50D2, Q5 IXTP3N50D2, Q6 IXTP3N50D2, Q7 IXTP3N50D2, Q8 IXTP3N50D2, Q9 IXTP3N50D2, SW1 SW_Push, SW2 SW_Push, U1 ChinaBluePill, U2 uA7805, U3 ESP-01, U4 RS485_Transeiver

Commit message: New PCB 2.0
Routing:
- net Net-(J10-Pad2): track 117.9 -> 129.9 mm, vias 2 -> 1
- net Net-(Q1-Pad1): track 20.0 -> 11.5 mm
- net Net-(Q3-Pad1): track 13.9 -> 11.6 mm
- net /MODE_0: track 13.3 -> 11.1 mm, vias 1 -> 0
- net /PWM_CH2_R: track 57.1 -> 55.9 mm
- net /MODE_1: track 13.3 -> 12.2 mm, vias 1 -> 0
- net /WS2812_CH2: track 84.5 -> 83.9 mm
- net /BUTTON: track 71.3 -> 71.6 mm, vias 3 -> 2
- net /RS485_RXTX: track 23.0 -> 23.1 mm, vias 1 -> 0
- net /RS232_RX: vias 2 -> 1
- net /LED: vias 1 -> 0
- net /A1: vias 2 -> 1
